File: Airbrakes/EAGLE/project_ACE/ACE.sch (EAGLE design)
At the start: 1 part

Commit message: Update CAD with BNO08x, OpenLog
Parts:
- removed SV1: (no value), con-lstb:MA03-2
- added J2, J4: SMD, SparkFun-Connectors:QWIIC_CONNECTORJS-1MM
- added J3: PTH, SparkX:I2C_STANDARD_NO_SILK
- added J6: (no value), SparkFun-Connectors:CONN_06NO_SILK_NO_POP
- added JP1, JP2: (no value), microbuilder:HEADER-1X670MIL
- added PORTENTA_H7: ABX00042, ABX00042:ABX00042
Connections:
- new net 3.3V: J2.2, J3.VCC, J4.2, J6.3, JP1.2
- new net BOOT: JP2.1
- new net CS: JP2.6
- new net DTR: J6.6
- new net GND: J2.1, J3.GND, J4.1, J6.1, J6.2, JP1.3
- new net INT: JP1.6
- new net MOSI: JP2.5
- new net PS0: JP2.2
- new net PS1: JP2.3
- new net RST: JP2.4
- new net RXI: J6.4
- new net SCL: J2.4, J3.SCL, J4.4
- new net SCL/SCK/RX: JP1.4
- new net SDA: J2.3, J3.SDA, J4.3
- new net SDA/MISO/TX: JP1.5
- new net TXO: J6.5
- new net VCC: JP1.1
Other:
- note added: "BNO085 Comms Pinout"
- note added: "Note: Portenta H7 is not lite version. Should be fine, given only VIN, GND, and any serial comm/electromotive/analog IO will be used"
- note added: "OpenLog Comms Pinout"
