File: Airbrakes/EAGLE/project_ACE/ACEnewSensors.sch (EAGLE design)
At the start: 22 parts, among them J1 10118192-0002LF, J2 10118192-0002LF, J3 PTH, U1 MPM3630GQV-P

Commit message: WIP refactoring
Parts:
- removed 7.4POWER: 282837-2, 282837-2:282837-2
- added 7.4POWER_TERMINAL: 282837-2, 282837-2:282837-2
- renumbered J1 to CAM1, J2 to CAM2
Connections:
- net SERVO_PWM renamed SRV_PWM
- removed net N$4: C2.1, C2A.1, C4.2, CAM1.1, CAM2.1, R1.1, U$10.VIN, U1.OUT, U1.OUT_2, U1.OUT_3
- removed net SERVO_VIN: 7.4POWER.1, C1.2, R3.2, SERVOCON.1, U1.IN
- new net 5VO: C2.2, C2A.2, C4.2, CAM1.1, CAM2.1, R1.2, U$10.VIN, U1.OUT, U1.OUT_2, U1.OUT_3
- new net 7.4V: 7.4POWER_TERMINAL.1, C1.1, R3.2, SERVOCON.1, U1.IN
- net GND: now also C1.2, C2.1, C2A.1; no longer C1.1, C2.2, C2A.2
- net N$5: now also R5.2; no longer R5.1
- net N$7: now also R1.1; no longer R1.2
- net PWR_GD: now also R5.1; no longer R5.2
- net SERVO_GND: now also 7.4POWER_TERMINAL.2; no longer 7.4POWER.2
Other:
- note added: "NOTE: move rot switch between 7.4v line to turn on both servo and logic"
- moved on the sheet: C1, C2, C2A, C4, R1, R2, R3, R5, ROTARY_TERMINAL, SERVOCON

Commit message: First draft of PACE
Parts:
- removed 7.4POWER_TERMINAL, ROTARY_TERMINAL: 282837-2, 282837-2:282837-2
- removed C1, C2, C2A: CL31B226KPHNNNE, 22uF_Capacitor:CL31B226KPHNNNE
- removed R1: ERJ-3EKF5102V, 51kO_Resistor:ERJ-3EKF5102V
- removed R2: ERA3AEB6981V, 6_98kO_Resistor:ERA3AEB6981V
- removed R5: RC1005F103CS, 10kO_Resistor:RC1005F103CS
- removed U1: MPM3630GQV-P, MPM3630:MPM3630GQV-P
- added ACE_ROT3: 282837-2, 282837-2:282837-2
- added BATT_TERM: XT30PW-F, XT30PW-F:XT30PW-F
- added C2A1, C5: CL31B226KPHNNNE, 22uF_Capacitor:CL31B226KPHNNNE
- added C6: 885012005009, 22pF_Capacitor:885012005009
- added CAM3, CAM4: 10118194-0001LF, USB_Micro_B_v2:10118194-0001LF
- added R6: RM04F1003CT, 100kO_Resistor:RM04F1003CT
- added R7: ERA3AEB6981V, 6_98kO_Resistor:ERA3AEB6981V
- added R8: ERJ-3EKF5102V, 51kO_Resistor:ERJ-3EKF5102V
- added U2: MPM3630GQV-P, MPM3630:MPM3630GQV-P
- C4: value 885012005009 -> CL31B226KPHNNNE; device 22pF_Capacitor:885012005009 -> 22uF_Capacitor:CL31B226KPHNNNE
- CAM1, CAM2: value 10118192-0002LF -> 10118194-0001LF; device USB_Micro_B:10118192-0002LF -> USB_Micro_B_v2:10118194-0001LF
- R3: value RM04F1003CT -> RC1005F103CS; device 100kO_Resistor:RM04F1003CT -> 10kO_Resistor:RC1005F103CS
Connections:
- removed net 7.4V: 7.4POWER_TERMINAL.1, C1.1, R3.2, SERVOCON.1, U1.IN
- removed net N$3: R3.1, U1.EN/SYNC
- removed net N$5: R5.2, U1.VCC
- removed net N$7: C4.1, R1.1, R2.2, U1.FB
- removed net PWR_GD: R5.1, U1.PG
- removed net SERVO_GND: 7.4POWER_TERMINAL.2, ROTARY_TERMINAL.1
- new net 7.4VCC: ACE_ROT3.1, C5.1, R6.2, SERVOCON.1, U2.IN
- new net 7.4VIN: ACE_ROT3.2, BATT_TERM.P
- new net AGND: R7.1, U2.AGND
- new net EN: R6.1, U2.EN/SYNC
- new net FB: C6.1, R7.2, R8.1, U2.FB
- new net MPM_VCC: R3.2, U2.VCC
- new net PG: R3.1, U2.PG
- new net STAT_LED: U$10.PWM_7
- net 5VO: now also C2A1.2, C6.2, CAM3.1, CAM4.1, R8.2, U2.OUT, U2.OUT_2, U2.OUT_3; no longer C2.2, C2A.2, R1.2, U1.OUT, U1.OUT_2, U1.OUT_3
- net GND: now also BATT_TERM.N, C2A1.1, C4.1, C5.2, CAM3.5, CAM4.5, U2.PGND, U2.PGND_2, U2.PGND_3; no longer C1.2, C2.1, C2A.1, R2.1, ROTARY_TERMINAL.2, U1.AGND, U1.PGND
Other:
- note removed: "NOTE: move rot switch between 7.4v line to turn on both servo and logic"
