File: Airbrakes/EAGLE/project_ACE/ACEnewSensors.sch (EAGLE design)
At the start: 14 parts, among them J3 PTH

Commit message: Finalize v0.2 ACE PCB
Parts:
- removed R1: 0 ohm, fab_new:R1206
- removed R2, R3: (no value), fab_new:R1206
Connections:
- removed net 3.3V: J3.VCC, JP1.2, U$10.3V3
- removed net VIN: JP1.1
- net GND: no longer R1.1
- net N$2: now also JP1.2; no longer R2.2, R3.1
- net SDA: no longer R2.1, R3.2
- net SERVO_PWM: now also U$10.CLK; no longer U$10.PWM_7
- net VCC: now also J3.VCC, JP1.1, U$10.3V3; no longer U$10.+5V
Other:
- note added: "3Vo"

Commit message: Added MPM3630
Parts:
- added C1, C2, C2A, C2B: 22uF, ngspice-simulation:C
- added C3: 51K, ngspice-simulation:C
- added R1, R3: 51K, ngspice-simulation:R
- added R2: 76.8k, ngspice-simulation:R
- added R4: 100k, ngspice-simulation:R
- added R5: 10k, ngspice-simulation:R
- added U1: MPM3630GQV-P, MPM3630:MPM3630GQV-P
Connections:
- new net N$3: R4.1, U1.EN/SYNC
- new net N$4: C2.2, C2A.2, C2B.2, C3.2, R1.2, U$10.VIN, U1.OUT
- new net N$5: R5.1, U1.VCC
- new net N$6: R5.2, U1.PG
- new net N$7: R3.1, U1.FB
- new net N$8: C3.1, R1.1, R2.1, R3.2
- net GND: now also C1.2, C2.1, C2A.1, C2B.1, R2.2, U1.AGND, U1.PGND
- net SERVO_VIN: now also C1.1, R4.2, U1.IN

Commit message: PACE Start
Parts:
- removed C2B: 22uF, ngspice-simulation:C
- removed C3: 51K, ngspice-simulation:C
- removed R4: 100k, ngspice-simulation:R
- removed SERVO: (no value), con-wago-508:W237-3E
- added C4: 885012005009, 22pF_Capacitor:885012005009
- added J1, J2: 10118192-0002LF, USB_Micro_B:10118192-0002LF
- added SERVOCON: B03B-PASK-1_(LF)_(SN), 3_Pin_JST_XA_Surface_Connector:B03B-PASK-1_(LF)_(SN)
- C1, C2, C2A: value 22uF -> CL31B226KPHNNNE; device ngspice-simulation:C -> 22uF_Capacitor:CL31B226KPHNNNE
- R1: value 51K -> ERJ-3EKF5102V; device ngspice-simulation:R -> 51kO_Resistor:ERJ-3EKF5102V
- R2: value 76.8k -> ERA3AEB6981V; device ngspice-simulation:R -> 6_98kO_Resistor:ERA3AEB6981V
- R3: value 51K -> RM04F1003CT; device ngspice-simulation:R -> 100kO_Resistor:RM04F1003CT
- R5: value 10k -> RC1005F103CS; device ngspice-simulation:R -> 10kO_Resistor:RC1005F103CS
Connections:
- net N$6 renamed PWR_GD
- removed net N$8: C3.1, R1.1, R2.1, R3.2
- net GND: now also C1.1, C2.2, C2A.2, J1.5, J2.5, R2.1, SERVOCON.2; no longer C1.2, C2.1, C2A.1, C2B.1, R2.2, SERVO-2.KL
- net N$3: now also R3.1; no longer R4.1
- net N$4: now also C2.1, C2A.1, C4.2, J1.1, J2.1, R1.1, U1.OUT_2, U1.OUT_3; no longer C2.2, C2A.2, C2B.2, C3.2, R1.2
- net N$7: now also C4.1, R1.2, R2.2; no longer R3.1
- net SERVO_PWM: now also SERVOCON.3; no longer SERVO-1.KL
- net SERVO_VIN: now also C1.2, R3.2, SERVOCON.1; no longer C1.1, R4.2, SERVO-3.KL

Commit message: First PACE layout draft (#98)
* WIP refactoring

* First draft of PACE

* Add MPM3630 block

* Finalize PACE board

* Add 51 Ohm resistor part

* Final revisions

---------

Co-authored-by: Breadn <bylueang@gmail.com>
Parts:
- removed 7.4POWER, ROTARY_TERMINAL: 282837-2, 282837-2:282837-2
- removed C1, C2, C2A: CL31B226KPHNNNE, 22uF_Capacitor:CL31B226KPHNNNE
- removed J1, J2: 10118192-0002LF, USB_Micro_B:10118192-0002LF
- removed R2: ERA3AEB6981V, 6_98kO_Resistor:ERA3AEB6981V
- removed R5: RC1005F103CS, 10kO_Resistor:RC1005F103CS
- removed U1: MPM3630GQV-P, MPM3630:MPM3630GQV-P
- added ACE_ROT3: 282837-2, 282837-2:282837-2
- added BATT_TERM: XT30PW-F, XT30PW-F:XT30PW-F
- added C2A1, C5: CL31B226KPHNNNE, 22uF_Capacitor:CL31B226KPHNNNE
- added C6: 885012005009, 22pF_Capacitor:885012005009
- added CAM1, CAM2, CAM3, CAM4: 10118194-0001LF, USB_Micro_B_v2:10118194-0001LF
- added R6: RM04F1003CT, 100kO_Resistor:RM04F1003CT
- added R7: ERA3AEB6981V, 6_98kO_Resistor:ERA3AEB6981V
- added R8: ERJ-3EKF5102V, 51kO_Resistor:ERJ-3EKF5102V
- added U2: MPM3630GQV-P, MPM3630:MPM3630GQV-P
- C4: value 885012005009 -> CL31B226KPHNNNE; device 22pF_Capacitor:885012005009 -> 22uF_Capacitor:CL31B226KPHNNNE
- R1: value ERJ-3EKF5102V -> ERJ3EKF51R0V; device 51kO_Resistor:ERJ-3EKF5102V -> ERJ3EKF51R0V-51Ohm-Resistor:ERJ3EKF51R0V
- R3: value RM04F1003CT -> RC1005F103CS; device 100kO_Resistor:RM04F1003CT -> 10kO_Resistor:RC1005F103CS
Connections:
- net SERVO_PWM renamed SRV_PWM
- removed net N$3: R3.1, U1.EN/SYNC
- removed net N$4: C2.1, C2A.1, C4.2, J1.1, J2.1, R1.1, U$10.VIN, U1.OUT, U1.OUT_2, U1.OUT_3
- removed net N$5: R5.1, U1.VCC
- removed net N$7: C4.1, R1.2, R2.2, U1.FB
- removed net PWR_GD: R5.2, U1.PG
- removed net SERVO_GND: 7.4POWER.2, ROTARY_TERMINAL.1
- removed net SERVO_VIN: 7.4POWER.1, C1.2, R3.2, SERVOCON.1, U1.IN
- new net 5VO: C2A1.2, C4.2, C6.2, CAM1.1, CAM2.1, CAM3.1, CAM4.1, R8.2, U$10.VIN, U2.OUT, U2.OUT_2, U2.OUT_3
- new net 7.4VCC: ACE_ROT3.1, C5.1, R6.2, SERVOCON.2, U2.IN
- new net 7.4VIN: ACE_ROT3.2, BATT_TERM.P
- new net AGND: R7.1, U2.AGND
- new net EN: R6.1, U2.EN/SYNC
- new net FB: C6.1, R7.2, R8.1, U2.FB
- new net LED: R1.2, U$10.PWM_7
- new net MPM_VCC: R3.2, U2.VCC
- new net PG: R3.1, U2.PG
- new net STAT_LED: R1.1
- net GND: now also BATT_TERM.N, C2A1.1, C4.1, C5.2, CAM1.5, CAM2.5, CAM3.5, CAM4.5, SERVOCON.1, U2.PGND, U2.PGND_2, U2.PGND_3; no longer C1.1, C2.2, C2A.2, J1.5, J2.5, R2.1, ROTARY_TERMINAL.2, SERVOCON.2, U1.AGND, U1.PGND
