File: Airbrakes/EAGLE/project_ACE/ACEnewSensors.brd (EAGLE design)
At the start: 114.5 x 63 mm, 33 parts, among them J3 PTH, U2 MPM3630GQV-P

Commit message: Finalize PACE board
Parts:
- added R1: ERJ3EKF51R0V, ERJ3EKF51R0V-51Ohm-Resistor:RES_ERJ3EKF51R0V
- moved CAM1 2.00 mm to (77.0, 6.69)
Connections:
- new net LED: R1.2, U$10.J9
- net 7.4VCC: now also SERVOCON.2; no longer SERVOCON.1
- net GND: now also SERVOCON.1; no longer SERVOCON.2
- net STAT_LED: now also R1.1; no longer U$10.J9
Routing:
- net STAT_LED: track 36.9 -> 3.26 mm, vias 3 -> 1
- net LED: track 0.00 -> 32.9 mm, vias 0 -> 1
- net 7.4VCC: track 41.3 -> 49.2 mm
- net 5VO: track 231.0 -> 234.1 mm, vias 17 -> 15
Other:
- board text removed: "NOTE: CHECK PIN ORDER ON EVERY TERMINAL (e.g. servo, batt term, etc.)"
