File: Airbrakes/EAGLE/project_ACE/ACEnewSensors.brd (EAGLE design)
At the start: 114.5 x 63 mm, 34 parts, among them J3 PTH, U2 MPM3630GQV-P

Commit message: Final revisions
Routing:
- net 7.4VCC: track 49.2 -> 51.7 mm
Changed lines of the file:
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@@
 <param name="rvMicroViaOuter" value="0.25"/>
 <param name="rvMicroViaInner" value="0.25"/>
-<param name="rlMinPadTop" value="10mil"/>
+<param name="rlMinPadTop" value="5mil"/>
 <param name="rlMaxPadTop" value="20mil"/>
 <param name="rlMinPadInner" value="10mil"/>
 <param name="rlMaxPadInner" value="20mil"/>
-<param name="rlMinPadBottom" value="10mil"/>
-<param name="rlMaxPadBottom" value="20mil"/>
-<param name="rlMinViaOuter" value="8mil"/>
+<param name="rlMinPadBottom" value="5mil"/>
+<param name="rlMaxPadBottom" value="50mil"/>
+<param name="rlMinViaOuter" value="7mil"/>
 <param name="rlMaxViaOuter" value="20mil"/>
-<param name="rlMinViaInner" value="8mil"/>
+<param name="rlMinViaInner" value="7mil"/>
 <param name="rlMaxViaInner" value="20mil"/>
 <param name="rlMinMicroViaOuter" value="4mil"/>
@@
 <wire x1="114.5" y1="42" x2="116.5066" y2="39.9934" width="1.27" layer="1"/>
 <wire x1="116.5066" y1="39.9934" x2="118.5" y2="39.9934" width="1.27" layer="1"/>
-<wire x1="110.838" y1="51.1058" x2="111.0539" y2="51.3217" width="0.508" layer="1"/>
+<wire x1="111.0539" y1="51.3217" x2="110.838" y2="51.1058" width="0.508" layer="1"/>
 <wire x1="111.0539" y1="51.3217" x2="111.0539" y2="52.245" width="0.508" layer="1"/>
-<wire x1="111.0539" y1="52.245" x2="113.245" y2="52.245" width="0.6096" layer="1"/>
+<wire x1="111.0539" y1="52.245" x2="111.5" y2="52.245" width="0.508" layer="1"/>
+<wire x1="111.5" y1="52.245" x2="112" y2="52.245" width="0.508" layer="1"/>
+<wire x1="112" y1="52.245" x2="112.5" y2="52.245" width="0.508" layer="1"/>
+<wire x1="112.5" y1="52.245" x2="113" y2="52.245" width="0.508" layer="1"/>
+<wire x1="113" y1="52.245" x2="113.245" y2="52.245" width="0.508" layer="1"/>
 <wire x1="113.3942" y1="51.1058" x2="114.3942" y2="51.1058" width="0.6096" layer="1"/>
 <wire x1="114.3942" y1="51.1058" x2="114.5" y2="51" width="0.6096" layer="1"/>
-<wire x1="113.245" y1="52.245" x2="114.5" y2="53.5" width="0.6096" layer="1"/>
+<wire x1="114.5" y1="53.5" x2="113.245" y2="52.245" width="0.6096" layer="1"/>
 <wire x1="113.3942" y1="51.1058" x2="114.5" y2="50" width="0.6096" layer="1"/>
 <wire x1="110.838" y1="51.1058" x2="113.3942" y2="51.1058" width="0.6096" layer="1"/>
 <wire x1="110.838" y1="51.1058" x2="111.2322" y2="51.5" width="0.6096" layer="1"/>
 <wire x1="114" y1="51.5" x2="114.5" y2="52" width="0.6096" layer="1"/>
-<wire x1="111.2322" y1="51.5" x2="114" y2="51.5" width="0.6096" layer="1"/>
-<wire x1="114.5" y1="52" x2="114.255" y2="52.245" width="0.6096" layer="1"/>
-<wire x1="114.255" y1="52.245" x2="113.245" y2="52.245" width="0.6096" layer="1"/>
-<wire x1="114.5" y1="52" x2="111.0666" y2="52" width="0.6096" layer="1"/>
+<wire x1="111.2322" y1="51.5" x2="112" y2="51.5" width="0.6096" layer="1"/>
+<wire x1="112" y1="51.5" x2="112.5" y2="51.5" width="0.6096" layer="1"/>
+<wire x1="112.5" y1="51.5" x2="113" y2="51.5" width="0.6096" layer="1"/>
+<wire x1="114" y1="51.5" x2="113.5" y2="51.5" width="0.6096" layer="1"/>
+<wire x1="113.5" y1="51.5" x2="113" y2="51.5" width="0.6096" layer="1"/>
+<wire x1="114" y1="52.245" x2="113.5" y2="52.245" width="0.6096" layer="1"/>
+<wire x1="113.245" y1="52.245" x2="113.5" y2="52.245" width="0.6096" layer="1"/>
+<wire x1="110.838" y1="51.1058" x2="111.5" y2="51.7678" width="0.508" layer="1"/>
+<wire x1="111.5" y1="51.7678" x2="111.5" y2="52.245" width="0.508" layer="1"/>
+<wire x1="112" y1="52.245" x2="112" y2="51.5" width="0.508" layer="1"/>
+<wire x1="112.5" y1="51.5" x2="112.5" y2="52.245" width="0.508" layer="1"/>
+<wire x1="113" y1="51.5" x2="113" y2="52" width="0.508" layer="1"/>
+<wire x1="113" y1="52" x2="113" y2="52.245" width="0.508" layer="1"/>
+<wire x1="113.5" y1="52.245" x2="113.5" y2="51.5" width="0.508" layer="1"/>
+<wire x1="114.5" y1="52" x2="114.255" y2="52.245" width="0.508" layer="1"/>
+<wire x1="114.255" y1="52.245" x2="114" y2="52.245" width="0.508" layer="1"/>
+<wire x1="114.5" y1="52" x2="113" y2="52" width="0.508" layer="1"/>
 </signal>
 <signal name="SRV_PWM">
@@
 <mfgpreviewcolor name="substratecolor" color="0xFF786E46"/>
 </mfgpreviewcolors>
+<errors>
+</errors>
 </board>
 </drawing>
