File: Airbrakes/EAGLE/project_PACE/PACE.sch (EAGLE design)
At the start: 22 parts, among them J3 PTH, U1 MPM3630GQV-P

Commit message: Add PACE project (#100)
* PACE Start

* First PACE layout draft (#98)

* WIP refactoring

* First draft of PACE

* Add MPM3630 block

* Finalize PACE board

* Add 51 Ohm resistor part

* Final revisions

---------

Co-authored-by: Breadn <bylueang@gmail.com>

* Reorganize local EAGLE files

* Reorganize PACE to new project folder

---------

Co-authored-by: wurdahl <44688469+wurdahl@users.noreply.github.com>
Co-authored-by: Breadn <bylueang@gmail.com>
Parts:
- removed 7.4POWER, ROTARY_TERMINAL: 282837-2, 282837-2:282837-2
- removed C1, C2, C2A, C2B: 22uF, ngspice-simulation:C
- removed C3: 51K, ngspice-simulation:C
- removed R2: 76.8k, ngspice-simulation:R
- removed R4: 100k, ngspice-simulation:R
- removed R5: 10k, ngspice-simulation:R
- removed SERVO: (no value), con-wago-508:W237-3E
- removed U1: MPM3630GQV-P, MPM3630:MPM3630GQV-P
- added ACE_ROT3: 282837-2, 282837-2:282837-2
- added BATT_TERM: XT30PW-F, XT30PW-F:XT30PW-F
- added C2A1, C4, C5: CL31B226KPHNNNE, 22uF_Capacitor:CL31B226KPHNNNE
- added C6: 885012005009, 22pF_Capacitor:885012005009
- added CAM1, CAM2, CAM3, CAM4: 10118194-0001LF, USB_Micro_B_v2:10118194-0001LF
- added R6: RM04F1003CT, 100kO_Resistor:RM04F1003CT
- added R7: ERA3AEB6981V, 6_98kO_Resistor:ERA3AEB6981V
- added R8: ERJ-3EKF5102V, 51kO_Resistor:ERJ-3EKF5102V
- added SERVOCON: B03B-PASK-1_(LF)_(SN), 3_Pin_JST_XA_Surface_Connector:B03B-PASK-1_(LF)_(SN)
- added U2: MPM3630GQV-P, MPM3630:MPM3630GQV-P
- R1: value 51K -> ERJ3EKF51R0V; device ngspice-simulation:R -> ERJ3EKF51R0V-51Ohm-Resistor:ERJ3EKF51R0V
- R3: value 51K -> RC1005F103CS; device ngspice-simulation:R -> 10kO_Resistor:RC1005F103CS
Connections:
- removed net N$3: R4.1, U1.EN/SYNC
- removed net N$4: C2.2, C2A.2, C2B.2, C3.2, R1.2, U$10.VIN, U1.OUT
- removed net N$5: R5.1, U1.VCC
- removed net N$6: R5.2, U1.PG
- removed net N$7: R3.1, U1.FB
- removed net N$8: C3.1, R1.1, R2.1, R3.2
- removed net SERVO_GND: 7.4POWER.2, ROTARY_TERMINAL.1
- removed net SERVO_PWM: SERVO-1.KL, U$10.CLK
- removed net SERVO_VIN: 7.4POWER.1, C1.1, R4.2, SERVO-3.KL, U1.IN
- new net 5VO: C2A1.2, C4.2, C6.2, CAM1.1, CAM2.1, CAM3.1, CAM4.1, R8.2, U$10.VIN, U2.OUT, U2.OUT_2, U2.OUT_3
- new net 7.4VCC: ACE_ROT3.1, C5.1, R6.2, SERVOCON.2, U2.IN
- new net 7.4VIN: ACE_ROT3.2, BATT_TERM.P
- new net AGND: R7.1, U2.AGND
- new net EN: R6.1, U2.EN/SYNC
- new net FB: C6.1, R7.2, R8.1, U2.FB
- new net LED: R1.2, U$10.PWM_7
- new net MPM_VCC: R3.2, U2.VCC
- new net PG: R3.1, U2.PG
- new net SRV_PWM: SERVOCON.3, U$10.CLK
- new net STAT_LED: R1.1
- net GND: now also BATT_TERM.N, C2A1.1, C4.1, C5.2, CAM1.5, CAM2.5, CAM3.5, CAM4.5, SERVOCON.1, U2.PGND, U2.PGND_2, U2.PGND_3; no longer C1.2, C2.1, C2A.1, C2B.1, R2.2, ROTARY_TERMINAL.2, SERVO-2.KL, U1.AGND, U1.PGND
