File: Airbrakes/ACE 3.0/RP2040_minimal_r2/RP2040_minimal_r2.kicad_sch (KiCad schematic)
At the start: 44 parts, among them J1 USB_B_Micro, J2 Conn_01x02, J3 Conn_02x18_Odd_Even, J4 Conn_02x18_Odd_Even, U1 NCP1117-3.3_SOT223, U2 W25Q128JVS, U3 RP2040, U4 BMI088, U5 BMP581, U6 BMM350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

Commit message: fix some labelling on schematic for ACE 3.0
Connections:
- net GPIO12 is gone; now on net INT1_ACCEL: J3.28 (Pin_28)
- net GPIO13 is gone; now on net INT2_ACCEL: J3.30 (Pin_30)
- net GPIO14 is gone; now on net INT3_GYRO: J3.32 (Pin_32)
- net GPIO15 is gone; now on net INT4_GYRO: J3.34 (Pin_34)
- net GPIO16 is gone; now on net INT_BARO: J4.27 (Pin_27)
- net GPIO17 is gone; now on net INT_MAG: J4.25 (Pin_25)
- net GPIO4 is gone; now on net SDA: J3.12 (Pin_12)
- net GPIO5 is gone; now on net SCL: J3.14 (Pin_14)
Changed lines of the file:
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@@
 		)
 	)
-	(label "GPIO17"
+	(label "INT_MAG"
 		(at 358.14 152.4 0)
 		(fields_autoplaced yes)
@@
 		)
 	)
-	(label "GPIO4"
+	(label "SDA"
 		(at 339.09 134.62 180)
 		(fields_autoplaced yes)
@@
 		)
 	)
-	(label "GPIO12"
+	(label "INT1_ACCEL"
 		(at 339.09 154.94 180)
 		(fields_autoplaced yes)
@@
 		)
 	)
-	(label "GPIO5"
+	(label "SCL"
 		(at 339.09 137.16 180)
 		(fields_autoplaced yes)
@@
 		)
 	)
-	(label "GPIO15"
+	(label "INT4_GYRO"
 		(at 339.09 162.56 180)
 		(fields_autoplaced yes)
@@
 		)
 	)
-	(label "GPIO16"
+	(label "INT_BARO"
 		(at 358.14 154.94 0)
 		(fields_autoplaced yes)
@@
 		)
 	)
-	(label "GPIO13"
+	(label "INT2_ACCEL"
 		(at 339.09 157.48 180)
 		(fields_autoplaced yes)
@@
 		)
 	)
-	(label "GPIO14"
+	(label "INT3_GYRO"
 		(at 339.09 160.02 180)
 		(fields_autoplaced yes)
