File: Airbrakes/ACE 3.0/RP2040_minimal_r2/RP2040_minimal_r2.kicad_pcb (KiCad board)
At the start: 2 copper layers, 52 x 51 mm, 45 parts, among them J1 USB_B_Micro, J2 Conn_01x02, J3 104031-0811, J4 Conn_02x18_Odd_Even, U1 NCP1117-3.3_SOT223, U2 W25Q128JVS, U3 RP2040, U4 BMI088, U5 BMP581, U6 BMM350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

Commit message: WIP wiring + DRC checks
Parts:
- moved R6 7.58 mm to (78.0, 106.5), turned to 0 degrees
Routing:
- net /SDA: track 0.00 -> 40.6 mm, vias 0 -> 2
- net /INT_MAG: track 19.4 -> 33.5 mm, vias 1 -> 2
- net +3V3: track 83.1 -> 69.3 mm, vias 3 -> 2
- net Net-(J3-CD/DAT3): track 1.79 -> 9.00 mm, vias 0 -> 2
- net GND: track 115.9 -> 112.2 mm, vias 31 -> 32
- net /SCL: track 0.00 -> 0.73 mm, vias 0 -> 1
- net /INT_BARO: track 34.9 -> 34.5 mm, vias 2 -> 1
