File: Airbrakes/KiCad/ACE 3.0/RP2040_minimal_r2/RP2040_minimal_r2.kicad_pcb (KiCad board)
At the start: 2 copper layers, 52 x 51 mm, 45 parts, among them J1 USB_B_Micro, J2 Conn_01x02, J3 104031-0811, J4 Conn_02x18_Odd_Even, U1 NCP1117-3.3_SOT223, U2 W25Q128JVS, U3 RP2040, U4 BMI088, U5 BMP581, U6 BMM350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

Commit message: Final routing draft + DRC fixes
Parts:
- moved C23 0.87 mm to (106.5, 116.3)
- moved C24 0.40 mm to (109.1, 118.1)
Routing:
- net /SCL: track 0.73 -> 42.5 mm, vias 1 -> 5
- net GND: track 112.2 -> 84.7 mm, vias 32 -> 34
- net +3V3: track 69.3 -> 45.1 mm
- net /INT_BARO: track 34.5 -> 28.3 mm, vias 1 -> 2
- net /SDA: track 40.6 -> 43.9 mm, vias 2 -> 3
- net /INT_MAG: track 33.5 -> 32.2 mm
- net /INT4_GYRO: track 18.9 -> 19.8 mm, vias 0 -> 4
- net /INT3_GYRO: track 17.7 -> 17.6 mm, vias 0 -> 4
Other:
- board text added: "BMI088"
- board text added: "BMM350"
- board text added: "BMP581"
- board text added: "Crystal"

Commit message: Silkscreen
Parts:
- added G***: LOGO, WURocketry_Logo:WURocketry_logo, F.Cu at (80.6, 81.7)
- added G***: LOGO, WURocketry_Logo:WURocketry_logo, B.Cu at (114.9, 87.2)
- moved C17 10.8 mm to (95.9, 78.4)
Other:
- board text added: "CORE"
- board text added: "CRYSTAL"
- board text added: "Courtesy of RP2040 Minimal Design, Raspberry Pi LTD https://datasheets.raspberrypi.com/rp2040/hardware-design-with-rp2040.pdf"
- board text added: "FLASH"
- board text added: "Inner Row GPIO Outer Row GND"
- board text added: "LDO"
- board text added: "SD & MMC"
- board text added: "WURocketry 2024-2025 @ Airbrakes / EE"
- board text added: "—{dblquote}Per Aspera Ad Astra{dblquote}"
- board text removed: "Crystal"
- board text removed: "Outer Row GND"
